File: front-panel.kicad_sch (KiCad schematic)
At the start: 36 parts, among them J1 PJ301M-12, J2 PJ301M-12, J3 PJ301M-12

Commit message: Version 1.3 of the model.
Parts:
- added D1: LED, eurocad:LED3mm, symbol Device:LED
- added R29: 1k_0603, Resistor_THT:R_Axial_DIN0207_L6.3mm_D2.5mm_P7.62mm_Horizontal, symbol PCM_4ms_Resistor:1k_0603
- gave numbers to parts that had none: 10
Connections:
- net Gate out: now also R29.1
- net Ground: now also D1.1 (K)
- new net: D1.2 (A), R29.2
